Commit message: fix tfs

File: auv_control_demos/chained_controllers/xacro/chained.urdf.xacro (robot description, xacro)
@@ -3,5 +3,5 @@
        name="auv">
   <link name="base_footprint" />
-  <link name="base_link">
+  <link name="base_link_auv">
     <origin xyz="0 0 0"
             rpy="0 0 0" />
@@ -45,5 +45,5 @@
             xyz="0 0 0" />
     <parent link="base_footprint" />
-    <child link="base_link" />
+    <child link="base_link_auv" />
   </joint>
   <!-- Thruster joints -->
@@ -53,5 +53,5 @@
     <origin rpy="-1.571 1.571 -0.785"
             xyz="0.14 -0.092 0.0" />
-    <parent link="base_link" />
+    <parent link="base_link_auv" />
     <child link="thruster_1" />
     <axis xyz="0 0 -1" />
@@ -62,5 +62,5 @@
     <origin rpy="-1.571 1.571 -2.356"
             xyz="0.14 0.092 0.0" />
-    <parent link="base_link" />
+    <parent link="base_link_auv" />
     <child link="thruster_2" />
     <axis xyz="0 0 -1" />
@@ -71,5 +71,5 @@
     <origin rpy="-1.571 1.571 0.785"
             xyz="-0.15 -0.092 0.0" />
-    <parent link="base_link" />
+    <parent link="base_link_auv" />
     <child link="thruster_3" />
     <axis xyz="0 0 -1" />
@@ -80,5 +80,5 @@
     <origin rpy="-1.571 1.571 2.356"
             xyz="-0.15 0.092 0.0" />
-    <parent link="base_link" />
+    <parent link="base_link_auv" />
     <child link="thruster_4" />
     <axis xyz="0 0 -1" />
@@ -89,5 +89,5 @@
     <origin rpy="0 0 0"
             xyz="0.118 -0.215 0.064" />
-    <parent link="base_link" />
+    <parent link="base_link_auv" />
     <child link="thruster_5" />
     <axis xyz="0 0 -1" />
@@ -98,5 +98,5 @@
     <origin rpy="0 0 0"
             xyz="0.118 0.215 0.064" />
-    <parent link="base_link" />
+    <parent link="base_link_auv" />
     <child link="thruster_6" />
     <axis xyz="0 0 -1" />
@@ -107,5 +107,5 @@
     <origin rpy="0 0 0"
             xyz="-0.118 -0.215 0.064" />
-    <parent link="base_link" />
+    <parent link="base_link_auv" />
     <child link="thruster_7" />
     <axis xyz="0 0 -1" />
@@ -116,5 +116,5 @@
     <origin rpy="0 0 0"
             xyz="-0.118 0.215 0.064" />
-    <parent link="base_link" />
+    <parent link="base_link_auv" />
     <child link="thruster_8" />
     <axis xyz="0 0 -1" />
